Commit message: wip

File: openarm_gripette_model/openarm_right/robot.urdf (robot description, URDF)
Before this commit: robot openarm_right, 13 links, 12 joints
Links:
- added link gripper, mass 1e-9
- link distal: mass 0.0471678 -> 0.0417207
- link feetech_sts3215__configuration_default: mass 0.101487 -> 0.100722
- link gripper_base: mass 0.213224 -> 0.208245
Joints:
- added joint gripper_frame: type fixed, parent gripper_base, child gripper, origin xyz=-0 0.1395 0.0305 rpy=-1.5708 1.5708 0, axis 0 0 0
- joint camera_frame: origin xyz=0.0687999 0.0662004 0.0260816 rpy=3.14159 1.57079 -1.5708 -> xyz=0.0689844 0.0662 0.0278102 rpy=-1.5708 1.5708 0
- joint distal: origin xyz=0.0249998 -0.0433013 -0.00055 rpy=0 0 2.0944 -> xyz=0.025 -0.0433013 -0.00055 rpy=0 0 2.0944
- joint proximal: limit lower=-1.57079 upper=7.64992e-06 effort=10 velocity=10 -> lower=-1.5708 upper=0 effort=10 velocity=10; origin xyz=0.0177499 0.1071 -0.0147625 rpy=1.5708 1.39626 -1.5708 -> xyz=0.0179344 0.1065 -0.0131898 rpy=1.5708 1.39626 -1.5708
- joint r_arm_pitch: limit lower=-2.99999 upper=0.999986 effort=10 velocity=10 -> lower=-2.96989 upper=1.0301 effort=10 velocity=10; origin xyz=-0 -0.0925 0.689 rpy=-1.5708 0 -0 -> xyz=-0 -0.0925 0.689 rpy=-1.5708 -0.0301087 -0
- joint r_arm_roll: limit lower=-3.31613 upper=0.174533 effort=10 velocity=10 -> lower=-3.33193 upper=0.158726 effort=10 velocity=10; origin xyz=-0.0301 0 -0.06 rpy=-3.14159 -1.5708 0 -> xyz=-0.0301 -0 -0.06 rpy=-1.5708 -1.55499 -1.5708
- joint r_arm_yaw: limit lower=-1.5708 upper=1.5708 effort=10 velocity=10 -> lower=-1.56755 upper=1.57405 effort=10 velocity=10
- joint r_elbow: origin xyz=0 -0.03155 -0.15375 rpy=-1.5708 -0 -0 -> xyz=-0.000102553 -0.0315498 -0.15375 rpy=-1.5708 -0 -0.00325049
- joint r_wrist_pitch: limit lower=-1.5708 upper=1.5708 effort=10 velocity=10 -> lower=-1.59567 upper=1.54592 effort=10 velocity=10; origin xyz=0.0205 -0 -0.0343 rpy=0 -1.5708 0 -> xyz=0.0205 -0 -0.0343 rpy=-1.5708 -1.54592 1.5708
- joint r_wrist_roll: limit lower=-0.785398 upper=0.785398 effort=10 velocity=10 -> lower=-0.796602 upper=0.774194 effort=10 velocity=10; origin xyz=0.0172 -0 -0.0455 rpy=-1.5708 -0 1.5708 -> xyz=0.0172 2.81739e-05 -0.0455 rpy=-1.5708 0.0112042 1.57243
- joint r_wrist_roll_mimic: origin xyz=0.0343 -0 -0.1205 rpy=-1.5708 0 -1.5708 -> xyz=0.0343 5.61841e-05 -0.1205 rpy=-1.5708 -0.0112042 -1.56916
- joint r_wrist_yaw: limit lower=-1.5708 upper=1.5708 effort=10 velocity=10 -> lower=-1.57243 upper=1.56916 effort=10 velocity=10

Commit message: update rotation axis

File: openarm_gripette_model/openarm_right/robot.urdf (robot description, URDF)
Before this commit: robot openarm_right, 14 links, 13 joints
Links:
- link distal: geometry collision mesh filename=package://assets/merged/distal_collision.stl; visual mesh filename=package://assets/merged/distal_visual.stl
- link dm_j4310_1_2_step: geometry collision mesh filename=package://assets/merged/dm_j4310_1_2_step_collision.stl; visual mesh filename=package://assets/merged/dm_j4310_1_2_step_visual.stl
- link dm_j4310_1_2_step_2: geometry collision mesh filename=package://assets/merged/dm_j4310_1_2_step_2_collision.stl; visual mesh filename=package://assets/merged/dm_j4310_1_2_step_2_visual.stl
- link dm_j4340_2_step: geometry collision mesh filename=package://assets/merged/dm_j4340_2_step_collision.stl; visual mesh filename=package://assets/merged/dm_j4340_2_step_visual.stl
- link dm_j8009p_2_step_1: geometry collision mesh filename=package://assets/merged/dm_j8009p_2_step_1_collision.stl; visual mesh filename=package://assets/merged/dm_j8009p_2_step_1_visual.stl
- link feetech_sts3215__configuration_default: geometry collision mesh filename=package://assets/merged/feetech_sts3215__configuration_defa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; visual mesh filename=package://assets/merged/feetech_sts3215__configuration_defa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
- link gripper_base: geometry collision mesh filename=package://assets/merged/gripper_base_collision.stl; visual mesh filename=package://assets/merged/gripper_base_visual.stl
- link hfsb6_6060_750_1_step: geometry collision mesh filename=package://assets/merged/hfsb6_6060_750_1_step_collision.stl; visual mesh filename=package://assets/merged/hfsb6_6060_750_1_step_visual.stl
- link j2_b_2_step: geometry collision mesh filename=package://assets/merged/j2_b_2_step_collision.stl; visual mesh filename=package://assets/merged/j2_b_2_step_visual.stl
- link j6_a_3_step: geometry collision mesh filename=package://assets/merged/j6_a_3_step_collision.stl; visual mesh filename=package://assets/merged/j6_a_3_step_visual.stl
- link j7_e_2_step: geometry collision mesh filename=package://assets/merged/j7_e_2_step_collision.stl; visual mesh filename=package://assets/merged/j7_e_2_step_visual.stl
Joints:
- joint r_arm_pitch: limit lower=-2.96989 upper=1.0301 effort=10 velocity=10 -> lower=-1.0301 upper=2.96989 effort=10 velocity=10; origin xyz=-0 -0.0925 0.689 rpy=-1.5708 -0.0301087 -0 -> xyz=-0 -0.0925 0.689 rpy=1.5708 -0.0301087 -0
- joint r_arm_roll: limit lower=-3.33193 upper=0.158726 effort=10 velocity=10 -> lower=-0.158726 upper=3.33193 effort=10 velocity=10; origin xyz=-0.0301 -0 -0.06 rpy=-1.5708 -1.55499 -1.5708 -> xyz=-0.0301 0 0.06 rpy=-1.5708 1.55499 1.5708
- joint r_arm_yaw: origin xyz=-0 -0.06625 0.0301 rpy=-1.5708 -1.5708 0 -> xyz=-0 0.06625 -0.0301 rpy=1.5708 1.5708 0
- joint r_elbow: limit lower=-2.44346 upper=0 effort=10 velocity=10 -> lower=-0 upper=2.44346 effort=10 velocity=10; origin xyz=-0.000102553 -0.0315498 -0.15375 rpy=-1.5708 -0 -0.00325049 -> xyz=-0.000102553 -0.0315498 -0.15375 rpy=1.5708 -0 -0.00325049
- joint r_wrist_roll: limit lower=-0.796602 upper=0.774194 effort=10 velocity=10 -> lower=-0.774194 upper=0.796602 effort=10 velocity=10; origin xyz=0.0172 2.81739e-05 -0.0455 rpy=-1.5708 0.0112042 1.57243 -> xyz=0.0172 2.81739e-05 -0.0455 rpy=1.5708 0.0112042 1.57243
- joint r_wrist_roll_mimic: mimic joint=r_wrist_roll multiplier=-1.0 -> joint=r_wrist_roll_inv multiplier=-1.0
- joint r_wrist_yaw: origin xyz=-0 0.0955 0.0315 rpy=1.5708 -0 0 -> xyz=-0 -0.0955 -0.0315 rpy=-1.5708 0 -0

Commit message: fix sign

File: openarm_gripette_model/openarm_right/robot.urdf (robot description, URDF)
Before this commit: robot robot, 14 links, 13 joints
Joints:
- joint r_wrist_roll: axis 0 0 1 -> 0 0 -1; limit lower=-0.774194 upper=0.796602 effort=10 velocity=10 -> lower=-0.796602 upper=0.774194 effort=10 velocity=10
- joint r_wrist_roll_mimic: mimic joint=r_wrist_roll_inv multiplier=-1.0 -> joint=r_wrist_roll_inv multiplier=1.0

Commit message: fix another wrong axis

File: openarm_gripette_model/openarm_right/robot.urdf (robot description, URDF)
Before this commit: robot robot, 14 links, 13 joints
Joints:
- joint r_wrist_yaw: axis 0 0 1 -> 0 0 -1; limit lower=-1.57243 upper=1.56916 effort=10 velocity=10 -> lower=-1.56916 upper=1.57243 effort=10 velocity=10

Commit message: wrist pitch

File: openarm_gripette_model/openarm_right/robot.urdf (robot description, URDF)
Before this commit: robot robot, 14 links, 13 joints
Joints:
- joint r_arm_yaw: axis 0 0 1 -> 0 0 -1; limit lower=-1.56755 upper=1.57405 effort=10 velocity=10 -> lower=-1.57405 upper=1.56755 effort=10 velocity=10
- joint r_wrist_pitch: axis 0 0 1 -> 0 0 -1; limit lower=-1.59567 upper=1.54592 effort=10 velocity=10 -> lower=-1.54592 upper=1.59567 effort=10 velocity=10
